File: pcb/Acondicionamiento.sch (KiCad schematic (older format))
At the start: 31 parts, among them U7 LM2903, U8 LM2903

Commit message: Colocados todos los componenetes en el area. A revisar
Parts:
- added C34, C35, C36, C37: 100n, Capacitors_SMD:C_0805, symbol C
- C32, C33: Ref_Proveedor (none) -> tme
Connections:
- net ENC1_A: now also C34.1
- net ENC1_B: now also C35.1
- net ENC2_A: now also C36.1
- net ENC2_B: now also C37.1
- net GND: now also C34.2, C35.2, C36.2, C37.2
Changed lines of the file:
@@
 F 6 "~" H 2550 1250 60  0001 C CNN "Potencia"
 F 7 "~" H 2550 1250 60  0001 C CNN "Tolerancia"
-F 8 "08055C104K4T2A" H 2550 1250 60  0001 C CNN "tme"
-F 9 "~" H 2550 1250 60  0001 C CNN "Ref_Proveedor"
+F 8 "~" H 2550 1250 60  0001 C CNN "Provedor"
+F 9 "tme" H 2550 1250 60  0001 C CNN "Ref_Proveedor"
+F 10 "08055C104K4T2A" H 2550 1250 60  0001 C CNN "tme"
 	1    2550 1250
 	1    0    0    -1
@@
 F 6 "~" H 6250 1250 60  0001 C CNN "Potencia"
 F 7 "~" H 6250 1250 60  0001 C CNN "Tolerancia"
-F 8 "08055C104K4T2A" H 6250 1250 60  0001 C CNN "tme"
-F 9 "~" H 6250 1250 60  0001 C CNN "Ref_Proveedor"
+F 8 "~" H 6250 1250 60  0001 C CNN "Provedor"
+F 9 "tme" H 6250 1250 60  0001 C CNN "Ref_Proveedor"
+F 10 "08055C104K4T2A" H 6250 1250 60  0001 C CNN "tme"
 	1    6250 1250
 	1    0    0    -1
@@
 Wire Wire Line
 	9250 3850 9250 3500
+Wire Wire Line
+	1500 6050 1500 5900
+Wire Wire Line
+	1500 6500 1500 6350
+$Comp
+L GND #PWR096
+U 1 1 577AF8F2
+P 1500 6500
+F 0 "#PWR096" H 1500 6250 50  0001 C CNN
+F 1 "GND" H 1505 6327 50  0000 C CNN
+F 2 "" H 1500 6500 50  0000 C CNN
+F 3 "" H 1500 6500 50  0000 C CNN
+	1    1500 6500
+	1    0    0    -1
+$EndComp
+Wire Wire Line
+	4000 6050 4000 5900
+Wire Wire Line
+	4000 6500 4000 6350
+$Comp
+L GND #PWR097
+U 1 1 577AFBD6
+P 4000 6500
+F 0 "#PWR097" H 4000 6250 50  0001 C CNN
+F 1 "GND" H 4005 6327 50  0000 C CNN
+F 2 "" H 4000 6500 50  0000 C CNN
+F 3 "" H 4000 6500 50  0000 C CNN
+	1    4000 6500
+	1    0    0    -1
+$EndComp
+Wire Wire Line
+	6550 5400 6550 5250
+Wire Wire Line
+	6550 5850 6550 5700
+$Comp
+L GND #PWR098
+U 1 1 577AFE78
+P 6550 5850
+F 0 "#PWR098" H 6550 5600 50  0001 C CNN
+F 1 "GND" H 6555 5677 50  0000 C CNN
+F 2 "" H 6550 5850 50  0000 C CNN
+F 3 "" H 6550 5850 50  0000 C CNN
+	1    6550 5850
+	1    0    0    -1
+$EndComp
+Wire Wire Line
+	9000 5400 9000 5250
+Wire Wire Line
+	9000 5850 9000 5700
+$Comp
+L GND #PWR099
+U 1 1 577AFFDE
+P 9000 5850
+F 0 "#PWR099" H 9000 5600 50  0001 C CNN
+F 1 "GND" H 9005 5677 50  0000 C CNN
+F 2 "" H 9000 5850 50  0000 C CNN
+F 3 "" H 9000 5850 50  0000 C CNN
+	1    9000 5850
+	1    0    0    -1
+$EndComp
+Connection ~ 9000 5250
+Connection ~ 1500 5900
+Connection ~ 6550 5250
+Connection ~ 2350 3500
+$Comp
+L C C34
+U 1 1 577B0FFF
+P 1500 6200
+F 0 "C34" H 1615 6246 50  0000 L CNN
+F 1 "100n" H 1615 6155 50  0000 L CNN
+F 2 "Capacitors_SMD:C_0805" H 1538 6050 50  0001 C CNN
+F 3 "" H 1500 6200 50  0000 C CNN
+F 4 "avx" H 1500 6200 60  0001 C CNN "Fabricante"
+F 5 "08055C104K4T2A" H 1500 6200 60  0001 C CNN "Ref"
+F 6 "~" H 1500 6200 60  0001 C CNN "Potencia"
+F 7 "~" H 1500 6200 60  0001 C CNN "Tolerancia"
+F 8 "~" H 1500 6200 60  0001 C CNN "Provedor"
+F 9 "tme" H 1500 6200 60  0001 C CNN "Ref_Proveedor"
+F 10 "08055C104K4T2A" H 1500 6200 60  0001 C CNN "tme"
+	1    1500 6200
+	1    0    0    -1
+$EndComp
+$Comp
+L C C35
+U 1 1 577B13D3
+P 4000 6200
+F 0 "C35" H 4115 6246 50  0000 L CNN
+F 1 "100n" H 4115 6155 50  0000 L CNN
+F 2 "Capacitors_SMD:C_0805" H 4038 6050 50  0001 C CNN
+F 3 "" H 4000 6200 50  0000 C CNN
+F 4 "avx" H 4000 6200 60  0001 C CNN "Fabricante"
+F 5 "08055C104K4T2A" H 4000 6200 60  0001 C CNN "Ref"
+F 6 "~" H 4000 6200 60  0001 C CNN "Potencia"
+F 7 "~" H 4000 6200 60  0001 C CNN "Tolerancia"
+F 8 "~" H 4000 6200 60  0001 C CNN "Provedor"
+F 9 "tme" H 4000 6200 60  0001 C CNN "Ref_Proveedor"
+F 10 "08055C104K4T2A" H 4000 6200 60  0001 C CNN "tme"
+	1    4000 6200
+	1    0    0    -1
+$EndComp
+$Comp
+L C C36
+U 1 1 577B14BA
+P 6550 5550
+F 0 "C36" H 6665 5596 50  0000 L CNN
+F 1 "100n" H 6665 5505 50  0000 L CNN
+F 2 "Capacitors_SMD:C_0805" H 6588 5400 50  0001 C CNN
+F 3 "" H 6550 5550 50  0000 C CNN
+F 4 "avx" H 6550 5550 60  0001 C CNN "Fabricante"
+F 5 "08055C104K4T2A" H 6550 5550 60  0001 C CNN "Ref"
+F 6 "~" H 6550 5550 60  0001 C CNN "Potencia"
+F 7 "~" H 6550 5550 60  0001 C CNN "Tolerancia"
+F 8 "~" H 6550 5550 60  0001 C CNN "Provedor"
+F 9 "tme" H 6550 5550 60  0001 C CNN "Ref_Proveedor"
+F 10 "08055C104K4T2A" H 6550 5550 60  0001 C CNN "tme"
+	1    6550 5550
+	1    0    0    -1
+$EndComp
+$Comp
+L C C37
+U 1 1 577B1650
+P 9000 5550
+F 0 "C37" H 9115 5596 50  0000 L CNN
+F 1 "100n" H 9115 5505 50  0000 L CNN
+F 2 "Capacitors_SMD:C_0805" H 9038 5400 50  0001 C CNN
+F 3 "" H 9000 5550 50  0000 C CNN
+F 4 "avx" H 9000 5550 60  0001 C CNN "Fabricante"
+F 5 "08055C104K4T2A" H 9000 5550 60  0001 C CNN "Ref"
+F 6 "~" H 9000 5550 60  0001 C CNN "Potencia"
+F 7 "~" H 9000 5550 60  0001 C CNN "Tolerancia"
+F 8 "~" H 9000 5550 60  0001 C CNN "Provedor"
+F 9 "tme" H 9000 5550 60  0001 C CNN "Ref_Proveedor"
+F 10 "08055C104K4T2A" H 9000 5550 60  0001 C CNN "tme"
+	1    9000 5550
+	1    0    0    -1
+$EndComp
+Connection ~ 4000 5900
 $EndSCHEMATC

Commit message: finalizado el posicionado sobre la pcb
Parts:
- U7, U8: footprint Housings_SOIC:SOIC-8_3.9x4.9mm_Pitch1.27mm -> Housings_SSOP:TSSOP-8_4.4x3mm_Pitch0.65mm
Changed lines of the file:
@@
 F 0 "U7" H 2400 2050 50  0000 L CNN
 F 1 "LM2903" H 2400 1750 50  0000 L CNN
-F 2 "Housings_SOIC:SOIC-8_3.9x4.9mm_Pitch1.27mm" H 2360 1900 50  0001 C CNN
+F 2 "Housings_SSOP:TSSOP-8_4.4x3mm_Pitch0.65mm" H 2360 1900 50  0001 C CNN
 F 3 "" H 2360 1900 50  0000 C CNN
 F 4 "ti" H 2300 1900 60  0001 C CNN "Fabricante"
@@
 	1150 2750 1150 2950
 $Comp
-L GND #PWR074
+L GND #PWR078
 U 1 1 576D5A93
 P 1150 2950
-F 0 "#PWR074" H 1150 2700 50  0001 C CNN
+F 0 "#PWR078" H 1150 2700 50  0001 C CNN
 F 1 "GND" H 1155 2777 50  0000 C CNN
 F 2 "" H 1150 2950 50  0000 C CNN
@@
 	1150 4500 1150 4700
 $Comp
-L GND #PWR075
+L GND #PWR079
 U 1 1 576D6058
 P 1150 4700
-F 0 "#PWR075" H 1150 4450 50  0001 C CNN
+F 0 "#PWR079" H 1150 4450 50  0001 C CNN
 F 1 "GND" H 1155 4527 50  0000 C CNN
 F 2 "" H 1150 4700 50  0000 C CNN
@@
 F 0 "U7" H 2400 3800 50  0000 L CNN
 F 1 "LM2903" H 2400 3500 50  0000 L CNN
-F 2 "Housings_SOIC:SOIC-8_3.9x4.9mm_Pitch1.27mm" H 2350 3650 50  0001 C CNN
+F 2 "Housings_SSOP:TSSOP-8_4.4x3mm_Pitch0.65mm" H 2350 3650 50  0001 C CNN
 F 3 "" H 2350 3650 50  0000 C CNN
 F 4 "ti" H 2300 3650 60  0001 C CNN "Fabricante"
@@
 $EndComp
 $Comp
-L GND #PWR076
+L GND #PWR080
 U 1 1 576D692F
 P 2600 2300
-F 0 "#PWR076" H 2600 2050 50  0001 C CNN
+F 0 "#PWR080" H 2600 2050 50  0001 C CNN
 F 1 "GND" H 2605 2127 50  0000 C CNN
 F 2 "" H 2600 2300 50  0000 C CNN
@@
 	2600 2250 2600 2300
 $Comp
-L GND #PWR077
+L GND #PWR081
 U 1 1 576D69E8
 P 2550 1500
-F 0 "#PWR077" H 2550 1250 50  0001 C CNN
+F 0 "#PWR081" H 2550 1250 50  0001 C CNN
 F 1 "GND" H 2555 1327 50  0000 C CNN
 F 2 "" H 2550 1500 50  0000 C CNN
@@
 	2300 900  2300 1600
 $Comp
-L +5V #PWR078
+L +5V #PWR082
 U 1 1 576D6A66
 P 2300 900
-F 0 "#PWR078" H 2300 750 50  0001 C CNN
+F 0 "#PWR082" H 2300 750 50  0001 C CNN
 F 1 "+5V" H 2315 1073 50  0000 C CNN
 F 2 "" H 2300 900 50  0000 C CNN
@@
 F 0 "U8" H 6100 2050 50  0000 L CNN
 F 1 "LM2903" H 6100 1750 50  0000 L CNN
-F 2 "Housings_SOIC:SOIC-8_3.9x4.9mm_Pitch1.27mm" H 6060 1900 50  0001 C CNN
+F 2 "Housings_SSOP:TSSOP-8_4.4x3mm_Pitch0.65mm" H 6060 1900 50  0001 C CNN
 F 3 "" H 6060 1900 50  0000 C CNN
 F 4 "ti" H 6000 1900 60  0001 C CNN "Fabricante"
@@
 	4850 2750 4850 2950
 $Comp
-L GND #PWR079
+L GND #PWR083
 U 1 1 576FA5D7
 P 4850 2950
-F 0 "#PWR079" H 4850 2700 50  0001 C CNN
+F 0 "#PWR083" H 4850 2700 50  0001 C CNN
 F 1 "GND" H 4855 2777 50  0000 C CNN
 F 2 "" H 4850 2950 50  0000 C CNN
@@
 	4850 4500 4850 4700
 $Comp
-L GND #PWR080
+L GND #PWR084
 U 1 1 576FA5F3
 P 4850 4700
-F 0 "#PWR080" H 4850 4450 50  0001 C CNN
+F 0 "#PWR084" H 4850 4450 50  0001 C CNN
 F 1 "GND" H 4855 4527 50  0000 C CNN
 F 2 "" H 4850 4700 50  0000 C CNN
@@
 F 0 "U8" H 6100 3800 50  0000 L CNN
 F 1 "LM2903" H 6100 3500 50  0000 L CNN
-F 2 "Housings_SOIC:SOIC-8_3.9x4.9mm_Pitch1.27mm" H 6050 3650 50  0001 C CNN
+F 2 "Housings_SSOP:TSSOP-8_4.4x3mm_Pitch0.65mm" H 6050 3650 50  0001 C CNN
 F 3 "" H 6050 3650 50  0000 C CNN
 F 4 "ti" H 6000 3650 60  0001 C CNN "Fabricante"
@@
 $EndComp
 $Comp
-L GND #PWR081
+L GND #PWR085
 U 1 1 576FA614
 P 6300 2300
-F 0 "#PWR081" H 6300 2050 50  0001 C CNN
+F 0 "#PWR085" H 6300 2050 50  0001 C CNN
 F 1 "GND" H 6305 2127 50  0000 C CNN
 F 2 "" H 6300 2300 50  0000 C CNN
@@
 	6300 2250 6300 2300
 $Comp
-L GND #PWR082
+L GND #PWR086
 U 1 1 576FA61D
 P 6250 1500
-F 0 "#PWR082" H 6250 1250 50  0001 C CNN
+F 0 "#PWR086" H 6250 1250 50  0001 C CNN
 F 1 "GND" H 6255 1327 50  0000 C CNN
 F 2 "" H 6250 1500 50  0000 C CNN
@@
 	6000 900  6000 1600
 $Comp
-L +5V #PWR083
+L +5V #PWR087
 U 1 1 576FA627
 P 6000 900
-F 0 "#PWR083" H 6000 750 50  0001 C CNN
+F 0 "#PWR087" H 6000 750 50  0001 C CNN
 F 1 "+5V" H 6015 1073 50  0000 C CNN
 F 2 "" H 6000 900 50  0000 C CNN
@@
 	9250 1500 9250 2300
 $Comp
-L +5V #PWR084
+L +5V #PWR088
 U 1 1 57705564
 P 9250 1500
-F 0 "#PWR084" H 9250 1350 50  0001 C CNN
+F 0 "#PWR088" H 9250 1350 50  0001 C CNN
 F 1 "+5V" H 9265 1673 50  0000 C CNN
 F 2 "" H 9250 1500 50  0000 C CNN
@@
 $EndComp
 $Comp
-L GND #PWR085
+L GND #PWR089
 U 1 1 57705FAF
 P 5100 6850
-F 0 "#PWR085" H 5100 6600 50  0001 C CNN
+F 0 "#PWR089" H 5100 6600 50  0001 C CNN
 F 1 "GND" H 5105 6677 50  0000 C CNN
 F 2 "" H 5100 6850 50  0000 C CNN
@@
 Connection ~ 2650 5600
 $Comp
-L GND #PWR086
+L GND #PWR090
 U 1 1 57706538
 P 2650 6800
-F 0 "#PWR086" H 2650 6550 50  0001 C CNN
+F 0 "#PWR090" H 2650 6550 50  0001 C CNN
 F 1 "GND" H 2655 6627 50  0000 C CNN
 F 2 "" H 2650 6800 50  0000 C CNN
@@
 $EndComp
 $Comp
-L GND #PWR087
+L GND #PWR091
 U 1 1 57707F5A
 P 10100 6200
-F 0 "#PWR087" H 10100 5950 50  0001 C CNN
+F 0 "#PWR091" H 10100 5950 50  0001 C CNN
 F 1 "GND" H 10105 6027 50  0000 C CNN
 F 2 "" H 10100 6200 50  0000 C CNN
@@
 Connection ~ 7650 4950
 $Comp
-L GND #PWR088
+L GND #PWR092
 U 1 1 57707F69
 P 7650 6150
-F 0 "#PWR088" H 7650 5900 50  0001 C CNN
+F 0 "#PWR092" H 7650 5900 50  0001 C CNN
 F 1 "GND" H 7655 5977 50  0000 C CNN
 F 2 "" H 7650 6150 50  0000 C CNN
@@
 Connection ~ 7900 4950
 $Comp
-L GND #PWR089
+L GND #PWR093
 U 1 1 5770B847
 P 7900 6150
-F 0 "#PWR089" H 7900 5900 50  0001 C CNN
+F 0 "#PWR093" H 7900 5900 50  0001 C CNN
 F 1 "GND" H 7905 5977 50  0000 C CNN
 F 2 "" H 7900 6150 50  0000 C CNN
@@
 	7900 5550 7900 6150
 $Comp
-L GND #PWR090
+L GND #PWR094
 U 1 1 5770B95B
 P 10350 6150
-F 0 "#PWR090" H 10350 5900 50  0001 C CNN
+F 0 "#PWR094" H 10350 5900 50  0001 C CNN
 F 1 "GND" H 10355 5977 50  0000 C CNN
 F 2 "" H 10350 6150 50  0000 C CNN
@@
 	5350 6200 5350 6850
 $Comp
-L GND #PWR091
+L GND #PWR095
 U 1 1 5770BE1B
 P 5350 6850
-F 0 "#PWR091" H 5350 6600 50  0001 C CNN
+F 0 "#PWR095" H 5350 6600 50  0001 C CNN
 F 1 "GND" H 5355 6677 50  0000 C CNN
 F 2 "" H 5350 6850 50  0000 C CNN
@@
 $EndComp
 $Comp
-L GND #PWR092
+L GND #PWR096
 U 1 1 5770C0A4
 P 2900 6800
-F 0 "#PWR092" H 2900 6550 50  0001 C CNN
+F 0 "#PWR096" H 2900 6550 50  0001 C CNN
 F 1 "GND" H 2905 6627 50  0000 C CNN
 F 2 "" H 2900 6800 50  0000 C CNN
@@
 Connection ~ 10150 1800
 $Comp
-L +24V #PWR093
+L +24V #PWR097
 U 1 1 576F44E4
 P 10150 1500
-F 0 "#PWR093" H 10150 1350 50  0001 C CNN
+F 0 "#PWR097" H 10150 1350 50  0001 C CNN
 F 1 "+24V" H 10165 1673 50  0000 C CNN
 F 2 "" H 10150 1500 50  0000 C CNN
@@
 $EndComp
 $Comp
-L VSS #PWR094
+L VSS #PWR098
 U 1 1 576F4819
 P 9250 3500
-F 0 "#PWR094" H 9250 3350 50  0001 C CNN
+F 0 "#PWR098" H 9250 3350 50  0001 C CNN
 F 1 "VSS" H 9267 3673 50  0000 C CNN
 F 2 "" H 9250 3500 50  0000 C CNN
@@
 $EndComp
 $Comp
-L +24V #PWR095
+L +24V #PWR099
 U 1 1 576F48DC
 P 10150 3500
-F 0 "#PWR095" H 10150 3350 50  0001 C CNN
+F 0 "#PWR099" H 10150 3350 50  0001 C CNN
 F 1 "+24V" H 10165 3673 50  0000 C CNN
 F 2 "" H 10150 3500 50  0000 C CNN
@@
 	1500 6500 1500 6350
 $Comp
-L GND #PWR096
+L GND #PWR0100
 U 1 1 577AF8F2
 P 1500 6500
-F 0 "#PWR096" H 1500 6250 50  0001 C CNN
+F 0 "#PWR0100" H 1500 6250 50  0001 C CNN
 F 1 "GND" H 1505 6327 50  0000 C CNN
 F 2 "" H 1500 6500 50  0000 C CNN
@@
 	4000 6500 4000 6350
 $Comp
-L GND #PWR097
+L GND #PWR0101
 U 1 1 577AFBD6
 P 4000 6500
-F 0 "#PWR097" H 4000 6250 50  0001 C CNN
+F 0 "#PWR0101" H 4000 6250 50  0001 C CNN
 F 1 "GND" H 4005 6327 50  0000 C CNN
 F 2 "" H 4000 6500 50  0000 C CNN
@@
 	6550 5850 6550 5700
 $Comp
-L GND #PWR098
+L GND #PWR0102
 U 1 1 577AFE78
 P 6550 5850
-F 0 "#PWR098" H 6550 5600 50  0001 C CNN
+F 0 "#PWR0102" H 6550 5600 50  0001 C CNN
 F 1 "GND" H 6555 5677 50  0000 C CNN
 F 2 "" H 6550 5850 50  0000 C CNN
@@
 	9000 5850 9000 5700
 $Comp
-L GND #PWR099
+L GND #PWR0103
 U 1 1 577AFFDE
 P 9000 5850
-F 0 "#PWR099" H 9000 5600 50  0001 C CNN
+F 0 "#PWR0103" H 9000 5600 50  0001 C CNN
 F 1 "GND" H 9005 5677 50  0000 C CNN
 F 2 "" H 9000 5850 50  0000 C CNN

Commit message: finalizado conexionado de pads
Changed lines of the file:
@@
 Connection ~ 1500 5900
 Connection ~ 6550 5250
-Connection ~ 2350 3500
 $Comp
 L C C34
