File: pcb/Pines_E_S.sch (KiCad schematic (older format))
At the start: 27 parts, among them P1 CONN_01X04, P10 CONN_01X04, P11 CONN_01X02, P12 CONN_01X03, P13 CONN_01X02, P14 USB_MINI, P15 CONN_01X02, P16 CONN_02X03, P2 CONN_01X04, P3 CONN_01X03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

Commit message: añadidos led para estado y alimentacion externa para salidas digitales
Parts:
- removed P15: CONN_01X02, PhoenixContact:PhoenixContact_MPT_0,5_3-2,54, symbol CONN_01X02
- added P15: CONN_01X03, PhoenixContact:PhoenixContact_MPT_0,5_3-2,54, symbol CONN_01X03
Connections:
- net DO1: now also P15.3 (P3)
- net DO2: now also P15.2 (P2)
- new net DO_COM: P15.1 (P1)
Changed lines of the file:
@@
 $EndComp
 $Comp
-L GND #PWR048
+L GND #PWR051
 U 1 1 5768B5F2
 P 9950 5050
-F 0 "#PWR048" H 9950 4800 50  0001 C CNN
+F 0 "#PWR051" H 9950 4800 50  0001 C CNN
 F 1 "GND" H 9955 4877 50  0000 C CNN
 F 2 "" H 9950 5050 50  0000 C CNN
@@
 $EndComp
 $Comp
-L +5V #PWR049
+L +5V #PWR052
 U 1 1 5768B612
 P 9950 4550
-F 0 "#PWR049" H 9950 4400 50  0001 C CNN
+F 0 "#PWR052" H 9950 4400 50  0001 C CNN
 F 1 "+5V" H 9965 4723 50  0000 C CNN
 F 2 "" H 9950 4550 50  0000 C CNN
@@
 	7600 2750 7600 3600
 $Comp
-L GND #PWR050
+L GND #PWR053
 U 1 1 5769A794
 P 7600 3600
-F 0 "#PWR050" H 7600 3350 50  0001 C CNN
+F 0 "#PWR053" H 7600 3350 50  0001 C CNN
 F 1 "GND" H 7605 3427 50  0000 C CNN
 F 2 "" H 7600 3600 50  0000 C CNN
@@
 	1750 2300 2250 2300
 $Comp
-L GND #PWR051
+L GND #PWR054
 U 1 1 576A5875
 P 2150 2550
-F 0 "#PWR051" H 2150 2300 50  0001 C CNN
+F 0 "#PWR054" H 2150 2300 50  0001 C CNN
 F 1 "GND" H 2155 2377 50  0000 C CNN
 F 2 "" H 2150 2550 50  0000 C CNN
@@
 $EndComp
 $Comp
-L +5V #PWR052
+L +5V #PWR055
 U 1 1 576A589D
 P 2050 1550
-F 0 "#PWR052" H 2050 1400 50  0001 C CNN
+F 0 "#PWR055" H 2050 1400 50  0001 C CNN
 F 1 "+5V" H 2065 1723 50  0000 C CNN
 F 2 "" H 2050 1550 50  0000 C CNN
@@
 	6600 1250 6600 1450
 $Comp
-L GND #PWR053
+L GND #PWR056
 U 1 1 576A7CA4
 P 6600 1450
-F 0 "#PWR053" H 6600 1200 50  0001 C CNN
+F 0 "#PWR056" H 6600 1200 50  0001 C CNN
 F 1 "GND" H 6605 1277 50  0000 C CNN
 F 2 "" H 6600 1450 50  0000 C CNN
@@
 	1800 5550 1800 5700
 $Comp
-L GND #PWR054
+L GND #PWR057
 U 1 1 576A878C
 P 1800 5700
-F 0 "#PWR054" H 1800 5450 50  0001 C CNN
+F 0 "#PWR057" H 1800 5450 50  0001 C CNN
 F 1 "GND" H 1800 5550 50  0000 C CNN
 F 2 "" H 1800 5700 50  0000 C CNN
@@
 	1800 6750 1800 6900
 $Comp
-L GND #PWR055
+L GND #PWR058
 U 1 1 576A8DE5
 P 1800 6900
-F 0 "#PWR055" H 1800 6650 50  0001 C CNN
+F 0 "#PWR058" H 1800 6650 50  0001 C CNN
 F 1 "GND" H 1800 6750 50  0000 C CNN
 F 2 "" H 1800 6900 50  0000 C CNN
@@
 	8200 3250 8200 3000
 $Comp
-L GND #PWR056
+L GND #PWR059
 U 1 1 576DD990
 P 8200 3250
-F 0 "#PWR056" H 8200 3000 50  0001 C CNN
+F 0 "#PWR059" H 8200 3000 50  0001 C CNN
 F 1 "GND" H 8205 3077 50  0000 C CNN
 F 2 "" H 8200 3250 50  0000 C CNN
@@
 $EndComp
 $Comp
-L GND #PWR057
+L GND #PWR060
 U 1 1 576DD9D4
 P 8750 3250
-F 0 "#PWR057" H 8750 3000 50  0001 C CNN
+F 0 "#PWR060" H 8750 3000 50  0001 C CNN
 F 1 "GND" H 8755 3077 50  0000 C CNN
 F 2 "" H 8750 3250 50  0000 C CNN
@@
 $EndComp
 $Comp
-L +5V #PWR058
+L +5V #PWR061
 U 1 1 576F71C4
 P 4600 1950
-F 0 "#PWR058" H 4600 1800 50  0001 C CNN
+F 0 "#PWR061" H 4600 1800 50  0001 C CNN
 F 1 "+5V" H 4615 2123 50  0000 C CNN
 F 2 "" H 4600 1950 50  0000 C CNN
@@
 Connection ~ 4600 2350
 $Comp
-L GND #PWR059
+L GND #PWR062
 U 1 1 576F7397
 P 4700 4550
-F 0 "#PWR059" H 4700 4300 50  0001 C CNN
+F 0 "#PWR062" H 4700 4300 50  0001 C CNN
 F 1 "GND" H 4705 4377 50  0000 C CNN
 F 2 "" H 4700 4550 50  0000 C CNN
@@
 ENC1_PWR
 $Comp
-L VSS #PWR060
+L VSS #PWR063
 U 1 1 576F2E08
 P 6500 1050
-F 0 "#PWR060" H 6500 900 50  0001 C CNN
+F 0 "#PWR063" H 6500 900 50  0001 C CNN
 F 1 "VSS" H 6517 1223 50  0000 C CNN
 F 2 "" H 6500 1050 50  0000 C CNN
@@
 	8300 1250 8300 1450
 $Comp
-L GND #PWR061
+L GND #PWR064
 U 1 1 576F4194
 P 8300 1450
-F 0 "#PWR061" H 8300 1200 50  0001 C CNN
+F 0 "#PWR064" H 8300 1200 50  0001 C CNN
 F 1 "GND" H 8305 1277 50  0000 C CNN
 F 2 "" H 8300 1450 50  0000 C CNN
@@
 	8200 1150 8200 1050
 $Comp
-L +24V #PWR062
+L +24V #PWR065
 U 1 1 576F41DA
 P 8200 1050
-F 0 "#PWR062" H 8200 900 50  0001 C CNN
+F 0 "#PWR065" H 8200 900 50  0001 C CNN
 F 1 "+24V" H 8215 1223 50  0000 C CNN
 F 2 "" H 8200 1050 50  0000 C CNN
@@
 Wire Wire Line
 	1750 3400 2250 3400
-$Comp
-L CONN_01X02 P15
-U 1 1 577B226D
-P 2450 3750
-F 0 "P15" H 2528 3791 50  0000 L CNN
-F 1 "CONN_01X02" H 2528 3700 50  0000 L CNN
-F 2 "PhoenixContact:PhoenixContact_MPT_0,5_3-2,54" H 2450 3750 50  0001 C CNN
-F 3 "" H 2450 3750 50  0000 C CNN
-F 4 "phoenix contact" H -2850 5950 60  0001 C CNN "Fabricante"
-F 5 "1803277 + 1803578" H -2850 5950 60  0001 C CNN "Ref"
-F 6 "~" H -2850 5950 60  0001 C CNN "Potencia"
-F 7 "~" H -2850 5950 60  0001 C CNN "Tolerancia"
-F 8 "tme" H -2850 5950 60  0001 C CNN "Provedor"
-F 9 "MC1.5/2-G-3.81" H -2850 5950 60  0001 C CNN "Ref_Proveedor"
-	1    2450 3750
-	1    0    0    -1
-$EndComp
-Text GLabel 1750 3700 0    60   Input ~ 0
+Text GLabel 1750 3900 0    60   Input ~ 0
 DO1
 Text GLabel 1750 3800 0    60   Input ~ 0
 DO2
 Wire Wire Line
-	1750 3700 2250 3700
+	1750 3900 2250 3900
 Wire Wire Line
 	2250 3800 1750 3800
+$Comp
+L CONN_01X03 P15
+U 1 1 57B44255
+P 2450 3800
+F 0 "P15" H 2528 3841 50  0000 L CNN
+F 1 "CONN_01X03" H 2528 3750 50  0000 L CNN
+F 2 "PhoenixContact:PhoenixContact_MPT_0,5_3-2,54" H 2450 3800 50  0001 C CNN
+F 3 "" H 2450 3800 50  0000 C CNN
+F 4 "phoenix contact" H 1000 3850 60  0001 C CNN "Fabricante"
+F 5 "1803280 + 1803581" H 1000 3850 60  0001 C CNN "Ref"
+F 6 "~" H 1000 3850 60  0001 C CNN "Potencia"
+F 7 "~" H 1000 3850 60  0001 C CNN "Tolerancia"
+F 8 "tme" H 1000 3850 60  0001 C CNN "Provedor"
+F 9 "MC1.5/3-G-3.81" H 1000 3850 60  0001 C CNN "Ref_Proveedor"
+	1    2450 3800
+	1    0    0    -1
+$EndComp
+Wire Wire Line
+	2250 3700 1750 3700
+Text GLabel 1750 3700 0    60   Output ~ 0
+DO_COM
 $EndSCHEMATC
